File: PCB/PCB.kicad_pcb (KiCad board)
At the start: 2 copper layers, 331.5 x 122.2 mm, 212 parts, among them J1 Conn_01x04, J2 USB_C_Receptacle_USB2.0_16P, J3 Conn_01x05, U1 XC6206PxxxMR, U2 SRV05-4, U3 RP2040, U4 W25Q128JVS, Y1 Crystal_GND24

Commit message: keyboard matrix done
Parts:
- J2: value USB_C_Receptacle_USB2.0_16P -> USB
- moved S4 0.37 mm to (172.4, 129.0)
Connections:
- U3 pad 11: C8 -> C9
- U3 pad 12: C9 -> C10
- U3 pad 13: C10 -> C11
- U3 pad 14: C11 -> C12
- U3 pad 15: C12 -> C13
- U3 pad 16: C13 -> C14
- U3 pad 17: C14 -> C15
- U3 pad 18: C15 -> R5
- U3 pad 2: C0 -> C6
- U3 pad 27: R0 -> C0
- U3 pad 28: R1 -> C1
- U3 pad 29: R2 -> C2
- U3 pad 3: C1 -> R4
- U3 pad 30: R3 -> C3
- U3 pad 31: R4 -> unconnected-(U3-GPIO20-Pad31)
- U3 pad 32: R5 -> unconnected-(U3-GPIO21-Pad32)
- U3 pad 36: unconnected-(U3-GPIO24-Pad36) -> R3
- U3 pad 4: C2 -> unconnected-(U3-GPIO2-Pad4)
- U3 pad 40: unconnected-(U3-GPIO28/ADC2-Pad40) -> C4
- U3 pad 41: unconnected-(U3-GPIO29/ADC3-Pad41) -> C5
- U3 pad 5: C3 -> R0
- U3 pad 6: C4 -> R1
- U3 pad 7: C5 -> R2
- U3 pad 8: C6 -> C7
- U3 pad 9: C7 -> C8
Routing:
- net R0: track 268.4 -> 548.8 mm, vias 0 -> 2
- net R1: track 314.4 -> 575.3 mm, vias 2 -> 4
- net R2: track 314.4 -> 569.5 mm
- net R3: track 314.4 -> 457.8 mm
- net C0: track 79.1 -> 217.5 mm, vias 0 -> 1
- net C1: track 110.9 -> 224.9 mm
- net C2: track 121.3 -> 211.0 mm, vias 0 -> 1
- net C3: track 116.8 -> 182.1 mm, vias 0 -> 1
- net R4: track 298.5 -> 325.0 mm
- net R5: track 320.7 -> 343.6 mm
- net C4: track 92.8 -> 114.9 mm, vias 0 -> 1
- net C5: track 110.3 -> 119.3 mm, vias 0 -> 1
- net C13: track 285.4 -> 284.7 mm
- net C8: track 166.5 -> 167.2 mm
- net C15: track 285.2 -> 284.5 mm
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