File: PCB/PCB.kicad_pcb (KiCad board)
At the start: 2 copper layers, 331.5 x 122.2 mm, 212 parts, among them J1 Conn_01x04, J2 USB, J3 Conn_01x05, U1 XC6206PxxxMR, U2 SRV05-4, U3 RP2040, U4 W25Q128JVS, Y1 Crystal_GND24

Commit message: gerbers + bom + position files
Parts:
- J2: value USB -> USB_C_Receptacle_USB2.0_16P
Changed lines of the file:
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@@
 		(grid_origin 146.647 120.612)
 		(pcbplotparams
-			(layerselection 0x00000000_00000000_55555555_5755f5ff)
+			(layerselection 0x00000000_00000000_55555555_575555ff)
 			(plot_on_all_layers_selection 0x00000000_00000000_00000000_00000000)
 			(disableapertmacros no)
@@
 			(sketchdnponfab yes)
 			(crossoutdnponfab yes)
-			(subtractmaskfromsilk no)
+			(subtractmaskfromsilk yes)
 			(outputformat 1)
 			(mirror no)
-			(drillshape 1)
+			(drillshape 0)
 			(scaleselection 1)
-			(outputdirectory "")
+			(outputdirectory "Gerbers/")
 		)
 	)
@@
 			)
 		)
-		(property "Value" "USB"
+		(property "Value" "USB_C_Receptacle_USB2.0_16P"
 			(at 0.12175 0.62775 0)
 			(layer "F.Fab")
