File: PCB/PCB.kicad_pcb (KiCad board)
At the start: 2 copper layers, 331.5 x 122.2 mm, 212 parts, among them J1 Conn_01x04, J2 USB_C_Receptacle_USB2.0_16P, J3 Conn_01x05, U1 XC6206PxxxMR, U2 SRV05-4, U3 RP2040, U4 W25Q128JVS, Y1 Crystal_GND24

Commit message: updates
Parts:
- S4: moved to B.Cu
- moved S1 0.80 mm to (308.1, 52.8)
- turned S4 to 0 degrees
Connections:
- U2 pad 4: unconnected-(U2-IO3-Pad4) -> D-
- U2 pad 6: D- -> unconnected-(U2-IO4-Pad6)
- U4 pad 4: unconnected-(U4-GND-Pad4) -> GND
Routing:
- net GND: track 142.0 -> 143.9 mm, vias 72 -> 73
- net D-: track 187.4 -> 186.9 mm
