File: PCB/PCB.kicad_sch (KiCad schematic)
At the start: 212 parts, among them J1 Conn_01x04, J2 USB_C_Receptacle_USB2.0_16P, J3 Conn_01x05, U1 XC6206PxxxMR, U2 SRV05-4, U3 RP2040, U4 W25Q128JVS, Y1 Crystal_GND24

Commit message: keyboard matrix done
Connections:
- net C0: now also U3.27 (GPIO16); no longer U3.2 (GPIO0)
- net C1: now also U3.28 (GPIO17); no longer U3.3 (GPIO1)
- net C10: now also U3.12 (GPIO9); no longer U3.13 (GPIO10)
- net C11: now also U3.13 (GPIO10); no longer U3.14 (GPIO11)
- net C12: now also U3.14 (GPIO11); no longer U3.15 (GPIO12)
- net C13: now also U3.15 (GPIO12); no longer U3.16 (GPIO13)
- net C14: now also U3.16 (GPIO13); no longer U3.17 (GPIO14)
- net C15: now also U3.17 (GPIO14); no longer U3.18 (GPIO15)
- net C2: now also U3.29 (GPIO18); no longer U3.4 (GPIO2)
- net C3: now also U3.30 (GPIO19); no longer U3.5 (GPIO3)
- net C4: now also U3.40 (GPIO28/ADC2); no longer U3.6 (GPIO4)
- net C5: now also U3.41 (GPIO29/ADC3); no longer U3.7 (GPIO5)
- net C6: now also U3.2 (GPIO0); no longer U3.8 (GPIO6)
- net C7: now also U3.8 (GPIO6); no longer U3.9 (GPIO7)
- net C8: now also U3.9 (GPIO7); no longer U3.11 (GPIO8)
- net C9: now also U3.11 (GPIO8); no longer U3.12 (GPIO9)
- net R0: now also U3.5 (GPIO3); no longer U3.27 (GPIO16)
- net R1: now also U3.6 (GPIO4); no longer U3.28 (GPIO17)
- net R2: now also U3.7 (GPIO5); no longer U3.29 (GPIO18)
- net R3: now also U3.36 (GPIO24); no longer U3.30 (GPIO19)
- net R4: now also U3.3 (GPIO1); no longer U3.31 (GPIO20)
- net R5: now also U3.18 (GPIO15); no longer U3.32 (GPIO21)

Commit message: updates
Connections:
- net D-: now also U2.4 (IO3); no longer U2.6 (IO4)
- net GND: now also U4.4 (GND)
Changed lines of the file:
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@@
 	)
 	(no_connect
-		(at 114.3 55.88)
+		(at 88.9 60.96)
 	)
 	(no_connect
-		(at 88.9 60.96)
+		(at 114.3 60.96)
 	)
 	(no_connect
@@
 	(wire
 		(pts
+			(xy 118.11 55.88) (xy 114.3 55.88)
+		)
+		(stroke
+			(width 0)
+			(type default)
+		)
+	)
+	(wire
+		(pts
 			(xy 218.44 193.04) (xy 218.44 194.31)
 		)
@@
 	(global_label "D-"
 		(shape input)
-		(at 114.3 60.96 0)
+		(at 118.11 55.88 0)
 		(fields_autoplaced yes)
 		(effects
@@
 		)
 		(property "Intersheetrefs" "${INTERSHEET_REFS}"
-			(at 120.1276 60.96 0)
+			(at 123.9376 55.88 0)
 			(hide yes)
 			(show_name no)
@@
 					(unit 1)
 				)
+			)
+		)
+	)
+	(symbol
+		(lib_id "power:GND")
+		(at 50.8 275.59 0)
+		(unit 1)
+		(body_style 1)
+		(exclude_from_sim no)
+		(in_bom yes)
+		(on_board yes)
+		(in_pos_files yes)
+		(dnp no)
+		(fields_autoplaced yes)
+		(property "Reference" "#PWR029"
+			(at 50.8 281.94 0)
+			(hide yes)
+			(show_name no)
+			(do_not_autoplace no)
+			(effects
+				(font
+					(size 1.27 1.27)
+				)
+			)
+		)
+		(property "Value" "GND"
+			(at 50.8 280.67 0)
+			(show_name no)
+			(do_not_autoplace no)
+			(effects
+				(font
+					(size 1.27 1.27)
+				)
+			)
+		)
+		(property "Footprint" ""
+			(at 50.8 275.59 0)
+			(hide yes)
+			(show_name no)
+			(do_not_autoplace no)
+			(effects
+				(font
+					(size 1.27 1.27)
+				)
+			)
+		)
+		(property "Datasheet" ""
+			(at 50.8 275.59 0)
+			(hide yes)
+			(show_name no)
+			(do_not_autoplace no)
+			(effects
+				(font
+					(size 1.27 1.27)
+				)
+			)
+		)
+		(property "Description" "Power symbol creates a global label with name \"GND\" , ground"
+			(at 50.8 275.59 0)
+			(hide yes)
+			(show_name no)
+			(do_not_autoplace no)
+			(effects
+				(font
+					(size 1.27 1.27)
+				)
+			)
+		)
+		(pin "1"
+		)
+		(instances
+			(project "PCB"
+				(path "/8182a1ea-1f66-4a44-903d-a7ab5f38a699"
+					(reference "#PWR029")
+					(unit 1)
+				)
